File: CAD/HubsanTXModule/HubsanTXModule.brd (EAGLE design)
At the start: 100 x 80 mm, 13 parts, among them Q1 AO3404A, Q2 AO3404A

Commit message: name nets for RF
Connections:
- net 2 renamed UC_CS
- net 4 renamed UC_SCLK
- net 5 renamed UC_SDIO
Changed lines of the file:
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@@
 <wire x1="7.62" y1="30.48" x2="22.86" y2="30.48" width="0" layer="19" extent="1-1"/>
 </signal>
-<signal name="2">
+<signal name="UC_CS">
 <contactref element="J3" pad="8"/>
 <contactref element="U$1" pad="5"/>
@@
 <wire x1="7.62" y1="22.86" x2="5.08" y2="22.86" width="0" layer="19" extent="1-1"/>
 </signal>
-<signal name="4">
+<signal name="UC_SCLK">
 <contactref element="J3" pad="6"/>
 <contactref element="U$1" pad="7"/>
 <wire x1="7.62" y1="20.32" x2="5.08" y2="20.32" width="0" layer="19" extent="1-1"/>
 </signal>
-<signal name="5">
+<signal name="UC_SDIO">
 <contactref element="U$1" pad="8"/>
 <contactref element="J3" pad="5"/>

Commit message: more work on board
Parts:
- added C1: (no value), SparkFun-Capacitors:0805-CAP
- added C2: 100uF, SparkFun-Capacitors:NIC_10X10.5_CAP
- added JP1, JP2: (no value), pinhead:1X07M
Connections:
- removed net UC_CS: J3.8, U$1.5
- removed net UC_SCLK: J3.6, U$1.7
- removed net UC_SDIO: J3.5, U$1.8
- new net GIO1: JP1.2
- new net GIO2: JP1.4
- new net SCK: J3.6, JP2.2, U$1.7
- new net SCS: J3.8, JP2.3, U$1.5
- new net SDIO: J3.5, JP2.1, U$1.8
- net 3V3: now also C1.1, JP2.6
- net GND: now also C1.2, C2.-, JP1.7, JP2.5
- net JR_VBATT: now also C2.+
Changed lines of the file:
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@@
 </element>
 <element name="J5" library="SparkFun-Connectors" package="1X02" value="" x="30.48" y="34.29" rot="R90"/>
+<element name="JP1" library="pinhead" package="1X07M" value="" x="3.81" y="-15.24"/>
+<element name="JP2" library="pinhead" package="1X07M" value="" x="3.81" y="-21.59"/>
+<element name="C2" library="SparkFun-Capacitors" package="NIC_10X10.5_CAP" value="100uF" x="1.27" y="-33.02">
+<attribute name="PROD_ID" value="CAP-08362" x="1.27" y="-33.02" size="1.778" layer="27" display="off"/>
+</element>
+<element name="C1" library="SparkFun-Capacitors" package="0805-CAP" value="" x="-7.62" y="-35.56">
+<attribute name="PROD_ID" value="CAP-11330" x="-7.62" y="-35.56" size="1.778" layer="27" display="off"/>
+</element>
 </elements>
 <signals>
@@
 <contactref element="U$1" pad="23"/>
 <contactref element="J4" pad="2"/>
-<wire x1="5.08" y1="27.94" x2="29.21" y2="12.7" width="0" layer="19" extent="1-1"/>
-<wire x1="25.4" y1="33.02" x2="5.08" y2="27.94" width="0" layer="19" extent="1-1"/>
-<wire x1="17.78" y1="25.4" x2="5.08" y2="27.94" width="0" layer="19" extent="1-1"/>
-<wire x1="31.75" y1="12.7" x2="17.78" y2="25.4" width="0" layer="19" extent="1-1"/>
+<contactref element="JP1" pad="7"/>
+<contactref element="JP2" pad="5"/>
+<contactref element="C2" pad="-"/>
+<contactref element="C1" pad="2"/>
+<wire x1="22.86" y1="33.02" x2="25.4" y2="33.02" width="0" layer="19" extent="1-1"/>
+<wire x1="17.78" y1="25.4" x2="22.86" y2="33.02" width="0" layer="19" extent="1-1"/>
 <wire x1="7.62" y1="27.94" x2="17.78" y2="25.4" width="0" layer="19" extent="1-1"/>
-<wire x1="22.86" y1="33.02" x2="7.62" y2="27.94" width="0" layer="19" extent="1-1"/>
+<wire x1="5.08" y1="27.94" x2="7.62" y2="27.94" width="0" layer="19" extent="1-1"/>
+<wire x1="29.21" y1="12.7" x2="17.78" y2="25.4" width="0" layer="19" extent="1-1"/>
+<wire x1="31.75" y1="12.7" x2="29.21" y2="12.7" width="0" layer="19" extent="1-1"/>
+<wire x1="9.81" y1="-15.24" x2="29.21" y2="12.7" width="0" layer="19" extent="1-1"/>
+<wire x1="5.81" y1="-21.59" x2="9.81" y2="-15.24" width="0" layer="19" extent="1-1"/>
+<wire x1="-3.23" y1="-33.02" x2="5.81" y2="-21.59" width="0" layer="19" extent="1-1"/>
+<wire x1="-6.72" y1="-35.56" x2="-3.23" y2="-33.02" width="0" layer="19" extent="1-1"/>
 </signal>
 <signal name="JR_ANT">
@@
 <contactref element="R2" pad="1"/>
 <contactref element="R3" pad="1"/>
-<wire x1="19.05" y1="29.63" x2="29.21" y2="10.16" width="0" layer="19" extent="1-1"/>
-<wire x1="11.43" y1="33.44" x2="19.05" y2="29.63" width="0" layer="19" extent="1-1"/>
-<wire x1="31.75" y1="10.16" x2="19.05" y2="29.63" width="0" layer="19" extent="1-1"/>
-<wire x1="12.7" y1="25.4" x2="31.75" y2="10.16" width="0" layer="19" extent="1-1"/>
+<contactref element="C2" pad="+"/>
+<wire x1="12.7" y1="25.4" x2="19.05" y2="29.63" width="0" layer="19" extent="1-1"/>
+<wire x1="11.43" y1="33.44" x2="12.7" y2="25.4" width="0" layer="19" extent="1-1"/>
+<wire x1="29.21" y1="10.16" x2="19.05" y2="29.63" width="0" layer="19" extent="1-1"/>
+<wire x1="31.75" y1="10.16" x2="29.21" y2="10.16" width="0" layer="19" extent="1-1"/>
+<wire x1="5.77" y1="-33.02" x2="29.21" y2="10.16" width="0" layer="19" extent="1-1"/>
 </signal>
 <signal name="3V3">
@@
 <contactref element="R1" pad="1"/>
 <contactref element="R4" pad="1"/>
+<contactref element="JP2" pad="6"/>
+<contactref element="C1" pad="1"/>
+<wire x1="22.86" y1="27.94" x2="25.4" y2="27.94" width="0" layer="19" extent="1-1"/>
+<wire x1="19.05" y1="33.44" x2="22.86" y2="27.94" width="0" layer="19" extent="1-1"/>
+<wire x1="16.24" y1="33.34" x2="19.05" y2="33.44" width="0" layer="19" extent="1-1"/>
 <wire x1="14.24" y1="31.43" x2="16.24" y2="33.34" width="0" layer="19" extent="1-1"/>
-<wire x1="25.4" y1="27.94" x2="16.24" y2="33.34" width="0" layer="19" extent="1-1"/>
 <wire x1="11.43" y1="31.33" x2="14.24" y2="31.43" width="0" layer="19" extent="1-1"/>
-<wire x1="19.05" y1="33.44" x2="11.43" y2="31.33" width="0" layer="19" extent="1-1"/>
-<wire x1="15.24" y1="25.4" x2="25.4" y2="27.94" width="0" layer="19" extent="1-1"/>
-<wire x1="22.86" y1="27.94" x2="15.24" y2="25.4" width="0" layer="19" extent="1-1"/>
+<wire x1="15.24" y1="25.4" x2="14.24" y2="31.43" width="0" layer="19" extent="1-1"/>
+<wire x1="7.81" y1="-21.59" x2="15.24" y2="25.4" width="0" layer="19" extent="1-1"/>
+<wire x1="-8.52" y1="-35.56" x2="7.81" y2="-21.59" width="0" layer="19" extent="1-1"/>
 </signal>
 <signal name="TX">
@@
 <wire x1="7.62" y1="30.48" x2="22.86" y2="30.48" width="0" layer="19" extent="1-1"/>
 </signal>
-<signal name="UC_CS">
-<contactref element="J3" pad="8"/>
-<contactref element="U$1" pad="5"/>
-<wire x1="7.62" y1="25.4" x2="5.08" y2="25.4" width="0" layer="19" extent="1-1"/>
-</signal>
 <signal name="UC_PPM">
 <contactref element="U$1" pad="6"/>
@@
 <wire x1="7.62" y1="22.86" x2="5.08" y2="22.86" width="0" layer="19" extent="1-1"/>
 </signal>
-<signal name="UC_SCLK">
-<contactref element="J3" pad="6"/>
-<contactref element="U$1" pad="7"/>
-<wire x1="7.62" y1="20.32" x2="5.08" y2="20.32" width="0" layer="19" extent="1-1"/>
-</signal>
-<signal name="UC_SDIO">
-<contactref element="U$1" pad="8"/>
-<contactref element="J3" pad="5"/>
-<wire x1="7.62" y1="17.78" x2="5.08" y2="17.78" width="0" layer="19" extent="1-1"/>
-</signal>
 <signal name="7">
 <contactref element="U$1" pad="10"/>
@@
 <wire x1="11.43" y1="35.14" x2="14.14" y2="34.29" width="0" layer="19" extent="1-1"/>
 </signal>
+<signal name="GIO1">
+<contactref element="JP1" pad="2"/>
+</signal>
+<signal name="GIO2">
+<contactref element="JP1" pad="4"/>
+</signal>
+<signal name="SDIO">
+<contactref element="JP2" pad="1"/>
+<contactref element="U$1" pad="8"/>
+<contactref element="J3" pad="5"/>
+<wire x1="5.08" y1="17.78" x2="7.62" y2="17.78" width="0" layer="19" extent="1-1"/>
+<wire x1="-2.19" y1="-21.59" x2="5.08" y2="17.78" width="0" layer="19" extent="1-1"/>
+</signal>
+<signal name="SCK">
+<contactref element="JP2" pad="2"/>
+<contactref element="J3" pad="6"/>
+<contactref element="U$1" pad="7"/>
+<wire x1="5.08" y1="20.32" x2="7.62" y2="20.32" width="0" layer="19" extent="1-1"/>
+<wire x1="-0.19" y1="-21.59" x2="5.08" y2="20.32" width="0" layer="19" extent="1-1"/>
+</signal>
+<signal name="SCS">
+<contactref element="JP2" pad="3"/>
+<contactref element="J3" pad="8"/>
+<contactref element="U$1" pad="5"/>
+<wire x1="5.08" y1="25.4" x2="7.62" y2="25.4" width="0" layer="19" extent="1-1"/>
+<wire x1="1.81" y1="-21.59" x2="5.08" y2="25.4" width="0" layer="19" extent="1-1"/>
+</signal>
 </signals>

Commit message: update
Parts:
- removed JP1, JP2: (no value), pinhead:1X07M
- added U$3: A7105_DEVBOARD, rf:A7105_DEV1
- moved U$2 66.5 mm to (63.5, 67.3)
- moved Q1 16.7 mm to (12.7, 50.8)
- moved R3 16.7 mm to (8.89, 50.8)
- moved R4 16.7 mm to (16.5, 50.8)
- moved Q2 15.5 mm to (12.7, 45.7)
- moved R1 15.5 mm to (8.89, 45.7)
- moved R2 15.5 mm to (16.5, 45.7)
- moved J5 7.73 mm to (29.2, 41.9)
Connections:
- net 3V3: now also U$3.13; no longer JP2.6
- net GIO1: now also U$3.2; no longer JP1.2
- net GIO2: now also U$3.4; no longer JP1.4
- net GND: now also U$3.12, U$3.7; no longer JP1.7, JP2.5
- net SCK: now also U$3.9; no longer JP2.2
- net SCS: now also U$3.10; no longer JP2.3
- net SDIO: now also U$3.8; no longer JP2.1
