File: CAD/HubsanTXModule/HubsanTXModule.sch (EAGLE design)
At the start: 13 parts, among them Q1 AO3404A, Q2 AO3404A

Commit message: name nets for RF
Connections:
- net 2 renamed UC_CS
- net 4 renamed UC_SCLK
- net 5 renamed UC_SDIO
Changed lines of the file:
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@@
 <setting verticaltext="up"/>
 </settings>
-<grid distance="0.1" unitdist="inch" unit="inch" style="lines" multiple="1" display="yes" altdistance="0.01" altunitdist="inch" altunit="inch"/>
+<grid distance="0.1" unitdist="inch" unit="inch" style="lines" multiple="1" display="no" altdistance="0.01" altunitdist="inch" altunit="inch"/>
 <layers>
-<layer number="1" name="Top" color="4" fill="1" visible="yes" active="no"/>
-<layer number="16" name="Bottom" color="1" fill="1" visible="yes" active="no"/>
-<layer number="17" name="Pads" color="2" fill="1" visible="yes" active="no"/>
-<layer number="18" name="Vias" color="2" fill="1" visible="yes" active="no"/>
-<layer number="19" name="Unrouted" color="6" fill="1" visible="yes" active="no"/>
-<layer number="20" name="Dimension" color="15" fill="1" visible="yes" active="no"/>
-<layer number="21" name="tPlace" color="7" fill="1" visible="yes" active="no"/>
-<layer number="22" name="bPlace" color="7" fill="1" visible="yes" active="no"/>
-<layer number="23" name="tOrigins" color="15" fill="1" visible="yes" active="no"/>
-<layer number="24" name="bOrigins" color="15" fill="1" visible="yes" active="no"/>
-<layer number="25" name="tNames" color="7" fill="1" visible="yes" active="no"/>
-<layer number="26" name="bNames" color="7" fill="1" visible="yes" active="no"/>
-<layer number="27" name="tValues" color="7" fill="1" visible="yes" active="no"/>
-<layer number="28" name="bValues" color="7" fill="1" visible="yes" active="no"/>
+<layer number="1" name="Top" color="4" fill="1" visible="no" active="no"/>
+<layer number="16" name="Bottom" color="1" fill="1" visible="no" active="no"/>
+<layer number="17" name="Pads" color="2" fill="1" visible="no" active="no"/>
+<layer number="18" name="Vias" color="2" fill="1" visible="no" active="no"/>
+<layer number="19" name="Unrouted" color="6" fill="1" visible="no" active="no"/>
+<layer number="20" name="Dimension" color="15" fill="1" visible="no" active="no"/>
+<layer number="21" name="tPlace" color="7" fill="1" visible="no" active="no"/>
+<layer number="22" name="bPlace" color="7" fill="1" visible="no" active="no"/>
+<layer number="23" name="tOrigins" color="15" fill="1" visible="no" active="no"/>
+<layer number="24" name="bOrigins" color="15" fill="1" visible="no" active="no"/>
+<layer number="25" name="tNames" color="7" fill="1" visible="no" active="no"/>
+<layer number="26" name="bNames" color="7" fill="1" visible="no" active="no"/>
+<layer number="27" name="tValues" color="7" fill="1" visible="no" active="no"/>
+<layer number="28" name="bValues" color="7" fill="1" visible="no" active="no"/>
 <layer number="29" name="tStop" color="7" fill="3" visible="no" active="no"/>
 <layer number="30" name="bStop" color="7" fill="6" visible="no" active="no"/>
@@
 <layer number="35" name="tGlue" color="7" fill="4" visible="no" active="no"/>
 <layer number="36" name="bGlue" color="7" fill="5" visible="no" active="no"/>
-<layer number="37" name="tTest" color="7" fill="1" visible="yes" active="no"/>
-<layer number="38" name="bTest" color="7" fill="1" visible="yes" active="no"/>
+<layer number="37" name="tTest" color="7" fill="1" visible="no" active="no"/>
+<layer number="38" name="bTest" color="7" fill="1" visible="no" active="no"/>
 <layer number="39" name="tKeepout" color="4" fill="11" visible="no" active="no"/>
 <layer number="40" name="bKeepout" color="1" fill="11" visible="no" active="no"/>
@@
 <layer number="44" name="Drills" color="7" fill="1" visible="no" active="no"/>
 <layer number="45" name="Holes" color="7" fill="1" visible="no" active="no"/>
-<layer number="46" name="Milling" color="3" fill="1" visible="yes" active="no"/>
-<layer number="47" name="Measures" color="7" fill="1" visible="yes" active="no"/>
-<layer number="48" name="Document" color="7" fill="1" visible="yes" active="no"/>
-<layer number="49" name="Reference" color="7" fill="1" visible="yes" active="no"/>
-<layer number="50" name="dxf" color="7" fill="1" visible="yes" active="no"/>
-<layer number="51" name="tDocu" color="7" fill="1" visible="yes" active="no"/>
-<layer number="52" name="bDocu" color="7" fill="1" visible="yes" active="no"/>
-<layer number="53" name="tGND_GNDA" color="7" fill="9" visible="yes" active="no"/>
-<layer number="54" name="bGND_GNDA" color="1" fill="9" visible="yes" active="no"/>
-<layer number="56" name="wert" color="7" fill="1" visible="yes" active="no"/>
-<layer number="57" name="tCAD" color="7" fill="1" visible="yes" active="no"/>
-<layer number="59" name="tCarbon" color="7" fill="1" visible="yes" active="no"/>
-<layer number="60" name="bCarbon" color="7" fill="1" visible="yes" active="no"/>
+<layer number="46" name="Milling" color="3" fill="1" visible="no" active="no"/>
+<layer number="47" name="Measures" color="7" fill="1" visible="no" active="no"/>
+<layer number="48" name="Document" color="7" fill="1" visible="no" active="no"/>
+<layer number="49" name="Reference" color="7" fill="1" visible="no" active="no"/>
+<layer number="50" name="dxf" color="7" fill="1" visible="no" active="no"/>
+<layer number="51" name="tDocu" color="7" fill="1" visible="no" active="no"/>
+<layer number="52" name="bDocu" color="7" fill="1" visible="no" active="no"/>
+<layer number="53" name="tGND_GNDA" color="7" fill="9" visible="no" active="no"/>
+<layer number="54" name="bGND_GNDA" color="1" fill="9" visible="no" active="no"/>
+<layer number="56" name="wert" color="7" fill="1" visible="no" active="no"/>
+<layer number="57" name="tCAD" color="7" fill="1" visible="no" active="no"/>
+<layer number="59" name="tCarbon" color="7" fill="1" visible="no" active="no"/>
+<layer number="60" name="bCarbon" color="7" fill="1" visible="no" active="no"/>
 <layer number="90" name="Modules" color="5" fill="1" visible="yes" active="yes"/>
 <layer number="91" name="Nets" color="2" fill="1" visible="yes" active="yes"/>
@@
 </segment>
 </net>
-<net name="2" class="0">
+<net name="UC_CS" class="0">
 <segment>
 <pinref part="J3" gate="G$1" pin="8"/>
@@
 </segment>
 </net>
-<net name="4" class="0">
+<net name="UC_SCLK" class="0">
 <segment>
 <pinref part="J3" gate="G$1" pin="6"/>
@@
 </segment>
 </net>
-<net name="5" class="0">
+<net name="UC_SDIO" class="0">
 <segment>
 <pinref part="U$1" gate="G$1" pin="5"/>

Commit message: more work on board
Parts:
- added C1: (no value), SparkFun-Capacitors:10UF10V10%(0805)
- added C2: 100uF, SparkFun-Capacitors:100UF-63V-20%(ELECT)
- added JP1, JP2: (no value), pinhead:PINHD-1X7M
Connections:
- removed net UC_CS: J3.8, U$1.2
- removed net UC_SCLK: J3.6, U$1.4
- removed net UC_SDIO: J3.5, U$1.5
- new net GIO1: JP1.2
- new net GIO2: JP1.4
- new net SCK: J3.6, JP2.2, U$1.4
- new net SCS: J3.8, JP2.3, U$1.2
- new net SDIO: J3.5, JP2.1, U$1.5
- net 3V3: now also C1.1, JP2.6
- net GND: now also C1.2, C2.-, JP1.7, JP2.5
- net JR_VBATT: now also C2.+
Changed lines of the file:
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@@
 <part name="R4" library="SparkFun-Resistors" deviceset="10KOHM-1/10W-1%(0603)" device="0603" value="10K"/>
 <part name="J5" library="SparkFun-Connectors" deviceset="M02" device="PTH"/>
+<part name="JP1" library="pinhead" deviceset="PINHD-1X7" device="M"/>
+<part name="JP2" library="pinhead" deviceset="PINHD-1X7" device="M"/>
+<part name="C2" library="SparkFun-Capacitors" deviceset="100UF-63V-20%(ELECT)" device="" value="100uF"/>
+<part name="C1" library="SparkFun-Capacitors" deviceset="10UF10V10%(0805)" device=""/>
 </parts>
 <sheets>
@@
 <instance part="R4" gate="G$1" x="63.5" y="60.96"/>
 <instance part="J5" gate="G$1" x="86.36" y="86.36" rot="R180"/>
+<instance part="JP1" gate="A" x="116.84" y="68.58"/>
+<instance part="JP2" gate="A" x="137.16" y="68.58"/>
+<instance part="C2" gate="G$1" x="7.62" y="38.1"/>
+<instance part="C1" gate="G$1" x="33.02" y="33.02"/>
 </instances>
 <busses>
@@
 <pinref part="U$2" gate="G$1" pin="GND"/>
 <wire x1="20.32" y1="35.56" x2="20.32" y2="30.48" width="0.1524" layer="91"/>
-<label x="20.32" y="27.94" size="1.778" layer="95"/>
+<pinref part="C2" gate="G$1" pin="-"/>
+<wire x1="7.62" y1="33.02" x2="7.62" y2="30.48" width="0.1524" layer="91"/>
+<wire x1="7.62" y1="30.48" x2="20.32" y2="30.48" width="0.1524" layer="91"/>
+<pinref part="C1" gate="G$1" pin="2"/>
+<wire x1="20.32" y1="30.48" x2="33.02" y2="30.48" width="0.1524" layer="91"/>
+<label x="20.32" y="30.48" size="1.778" layer="95" rot="MR180"/>
 </segment>
 <segment>
@@
 <label x="106.68" y="35.56" size="1.778" layer="95"/>
 </segment>
+<segment>
+<pinref part="JP1" gate="A" pin="7"/>
+<wire x1="106.68" y1="60.96" x2="114.3" y2="60.96" width="0.1524" layer="91"/>
+<label x="106.68" y="60.96" size="1.778" layer="95" rot="MR0"/>
+</segment>
+<segment>
+<pinref part="JP2" gate="A" pin="5"/>
+<wire x1="127" y1="66.04" x2="134.62" y2="66.04" width="0.1524" layer="91"/>
+<label x="127" y="66.04" size="1.778" layer="95" rot="MR0"/>
+</segment>
 </net>
 <net name="JR_ANT" class="0">
@@
 <pinref part="U$2" gate="G$1" pin="IN"/>
 <wire x1="7.62" y1="43.18" x2="12.7" y2="43.18" width="0.1524" layer="91"/>
-<label x="0" y="43.18" size="1.778" layer="95"/>
+<pinref part="C2" gate="G$1" pin="+"/>
+<wire x1="7.62" y1="43.18" x2="7.62" y2="40.64" width="0.1524" layer="91"/>
+<label x="7.62" y="43.18" size="1.778" layer="95" rot="MR0"/>
 </segment>
 <segment>
@@
 <pinref part="R2" gate="G$1" pin="1"/>
 <wire x1="12.7" y1="81.28" x2="15.24" y2="81.28" width="0.1524" layer="91"/>
-<label x="2.54" y="81.28" size="1.778" layer="95"/>
+<label x="12.7" y="81.28" size="1.778" layer="95" rot="MR0"/>
 </segment>
 <segment>
 <pinref part="R3" gate="G$1" pin="1"/>
 <wire x1="55.88" y1="81.28" x2="58.42" y2="81.28" width="0.1524" layer="91"/>
-<label x="45.72" y="81.28" size="1.778" layer="95"/>
+<label x="55.88" y="81.28" size="1.778" layer="95" rot="MR0"/>
 </segment>
 </net>
@@
 <wire x1="27.94" y1="43.18" x2="33.02" y2="43.18" width="0.1524" layer="91"/>
 <label x="33.02" y="43.18" size="1.778" layer="95"/>
+<pinref part="C1" gate="G$1" pin="1"/>
+<wire x1="33.02" y1="43.18" x2="33.02" y2="38.1" width="0.1524" layer="91"/>
 </segment>
 <segment>
@@
 <pinref part="R1" gate="G$1" pin="1"/>
 <wire x1="12.7" y1="60.96" x2="15.24" y2="60.96" width="0.1524" layer="91"/>
-<label x="7.62" y="60.96" size="1.778" layer="95"/>
+<label x="12.7" y="60.96" size="1.778" layer="95" rot="MR0"/>
 </segment>
 <segment>
 <pinref part="R4" gate="G$1" pin="1"/>
 <wire x1="55.88" y1="60.96" x2="58.42" y2="60.96" width="0.1524" layer="91"/>
-<label x="50.8" y="60.96" size="1.778" layer="95"/>
+<label x="55.88" y="60.96" size="1.778" layer="95" rot="MR0"/>
+</segment>
+<segment>
+<pinref part="JP2" gate="A" pin="6"/>
+<wire x1="127" y1="63.5" x2="134.62" y2="63.5" width="0.1524" layer="91"/>
+<label x="127" y="63.5" size="1.778" layer="95" rot="MR0"/>
 </segment>
 </net>
@@
 <wire x1="121.92" y1="33.02" x2="101.6" y2="33.02" width="0.1524" layer="91"/>
 <label x="106.68" y="33.02" size="1.778" layer="95"/>
-</segment>
-</net>
-<net name="UC_CS" class="0">
-<segment>
-<pinref part="J3" gate="G$1" pin="8"/>
-<pinref part="U$1" gate="G$1" pin="2"/>
-<wire x1="58.42" y1="27.94" x2="78.74" y2="27.94" width="0.1524" layer="91"/>
-<label x="60.96" y="27.94" size="1.778" layer="95"/>
 </segment>
 </net>
@@
 <wire x1="25.4" y1="60.96" x2="25.4" y2="55.88" width="0.1524" layer="91"/>
 <junction x="25.4" y="60.96"/>
-<label x="25.4" y="55.88" size="1.778" layer="95"/>
-</segment>
-</net>
-<net name="UC_SCLK" class="0">
-<segment>
-<pinref part="J3" gate="G$1" pin="6"/>
-<pinref part="U$1" gate="G$1" pin="4"/>
-<wire x1="58.42" y1="22.86" x2="78.74" y2="22.86" width="0.1524" layer="91"/>
-<label x="60.96" y="22.86" size="1.778" layer="95"/>
-</segment>
-</net>
-<net name="UC_SDIO" class="0">
-<segment>
-<pinref part="U$1" gate="G$1" pin="5"/>
-<pinref part="J3" gate="G$1" pin="5"/>
-<wire x1="78.74" y1="20.32" x2="58.42" y2="20.32" width="0.1524" layer="91"/>
-<label x="60.96" y="20.32" size="1.778" layer="95"/>
+<label x="25.4" y="55.88" size="1.778" layer="95" rot="MR180"/>
 </segment>
 </net>
@@
 </segment>
 </net>
+<net name="GIO1" class="0">
+<segment>
+<pinref part="JP1" gate="A" pin="2"/>
+<wire x1="114.3" y1="73.66" x2="106.68" y2="73.66" width="0.1524" layer="91"/>
+<label x="106.68" y="73.66" size="1.778" layer="95" rot="MR0"/>
+</segment>
+</net>
+<net name="GIO2" class="0">
+<segment>
+<pinref part="JP1" gate="A" pin="4"/>
+<wire x1="106.68" y1="68.58" x2="114.3" y2="68.58" width="0.1524" layer="91"/>
+<label x="106.68" y="68.58" size="1.778" layer="95" rot="MR0"/>
+</segment>
+</net>
+<net name="SDIO" class="0">
+<segment>
+<pinref part="JP2" gate="A" pin="1"/>
+<wire x1="127" y1="76.2" x2="134.62" y2="76.2" width="0.1524" layer="91"/>
+<label x="127" y="76.2" size="1.778" layer="95" rot="MR0"/>
+</segment>
+<segment>
+<pinref part="U$1" gate="G$1" pin="5"/>
+<pinref part="J3" gate="G$1" pin="5"/>
+<wire x1="78.74" y1="20.32" x2="58.42" y2="20.32" width="0.1524" layer="91"/>
+<label x="60.96" y="20.32" size="1.778" layer="95"/>
+</segment>
+</net>
+<net name="SCK" class="0">
+<segment>
+<pinref part="JP2" gate="A" pin="2"/>
+<wire x1="127" y1="73.66" x2="134.62" y2="73.66" width="0.1524" layer="91"/>
+<label x="127" y="73.66" size="1.778" layer="95" rot="MR0"/>
+</segment>
+<segment>
+<pinref part="J3" gate="G$1" pin="6"/>
+<pinref part="U$1" gate="G$1" pin="4"/>
+<wire x1="58.42" y1="22.86" x2="78.74" y2="22.86" width="0.1524" layer="91"/>
+<label x="60.96" y="22.86" size="1.778" layer="95"/>
+</segment>
+</net>
+<net name="SCS" class="0">
+<segment>
+<pinref part="JP2" gate="A" pin="3"/>
+<wire x1="127" y1="71.12" x2="134.62" y2="71.12" width="0.1524" layer="91"/>
+<label x="127" y="71.12" size="1.778" layer="95" rot="MR0"/>
+</segment>
+<segment>
+<pinref part="J3" gate="G$1" pin="8"/>
+<pinref part="U$1" gate="G$1" pin="2"/>
+<wire x1="58.42" y1="27.94" x2="78.74" y2="27.94" width="0.1524" layer="91"/>
+<label x="60.96" y="27.94" size="1.778" layer="95"/>
+</segment>
+</net>

Commit message: update
Parts:
- removed JP1, JP2: (no value), pinhead:PINHD-1X7M
- added U$3: A7105_DEVBOARD, rf:A7105_DEVBOARD
Connections:
- net 3V3: now also U$3.VDD; no longer JP2.6
- net GIO1: now also U$3.GIO1; no longer JP1.2
- net GIO2: now also U$3.GIO2; no longer JP1.4
- net GND: now also U$3.GND1, U$3.GND2; no longer JP1.7, JP2.5
- net SCK: now also U$3.SCK; no longer JP2.2
- net SCS: now also U$3.SCS; no longer JP2.3
- net SDIO: now also U$3.SDIO; no longer JP2.1
Changed lines of the file:
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@@
 <setting verticaltext="up"/>
 </settings>
-<grid distance="0.1" unitdist="inch" unit="inch" style="lines" multiple="1" display="no" altdistance="0.01" altunitdist="inch" altunit="inch"/>
+<grid distance="0.1" unitdist="inch" unit="inch" style="lines" multiple="1" display="yes" altdistance="0.01" altunitdist="inch" altunit="inch"/>
 <layers>
 <layer number="1" name="Top" color="4" fill="1" visible="no" active="no"/>
@@
 <part name="R4" library="SparkFun-Resistors" deviceset="10KOHM-1/10W-1%(0603)" device="0603" value="10K"/>
 <part name="J5" library="SparkFun-Connectors" deviceset="M02" device="PTH"/>
-<part name="JP1" library="pinhead" deviceset="PINHD-1X7" device="M"/>
-<part name="JP2" library="pinhead" deviceset="PINHD-1X7" device="M"/>
 <part name="C2" library="SparkFun-Capacitors" deviceset="100UF-63V-20%(ELECT)" device="" value="100uF"/>
 <part name="C1" library="SparkFun-Capacitors" deviceset="10UF10V10%(0805)" device=""/>
+<part name="U$3" library="rf" deviceset="A7105_DEVBOARD" device=""/>
 </parts>
 <sheets>
@@
 <instance part="R4" gate="G$1" x="63.5" y="60.96"/>
 <instance part="J5" gate="G$1" x="86.36" y="86.36" rot="R180"/>
-<instance part="JP1" gate="A" x="116.84" y="68.58"/>
-<instance part="JP2" gate="A" x="137.16" y="68.58"/>
 <instance part="C2" gate="G$1" x="7.62" y="38.1"/>
 <instance part="C1" gate="G$1" x="33.02" y="33.02"/>
+<instance part="U$3" gate="G$1" x="114.3" y="55.88"/>
 </instances>
 <busses>
@@
 </segment>
 <segment>
-<pinref part="JP1" gate="A" pin="7"/>
-<wire x1="106.68" y1="60.96" x2="114.3" y2="60.96" width="0.1524" layer="91"/>
-<label x="106.68" y="60.96" size="1.778" layer="95" rot="MR0"/>
-</segment>
-<segment>
-<pinref part="JP2" gate="A" pin="5"/>
-<wire x1="127" y1="66.04" x2="134.62" y2="66.04" width="0.1524" layer="91"/>
-<label x="127" y="66.04" size="1.778" layer="95" rot="MR0"/>
+<wire x1="109.22" y1="60.96" x2="104.14" y2="60.96" width="0.1524" layer="91"/>
+<wire x1="104.14" y1="60.96" x2="104.14" y2="58.42" width="0.1524" layer="91"/>
+<wire x1="104.14" y1="58.42" x2="109.22" y2="58.42" width="0.1524" layer="91"/>
+<wire x1="101.6" y1="58.42" x2="104.14" y2="58.42" width="0.1524" layer="91"/>
+<label x="101.6" y="58.42" size="1.778" layer="95" rot="MR0"/>
+<pinref part="U$3" gate="G$1" pin="GND2"/>
+<pinref part="U$3" gate="G$1" pin="GND1"/>
 </segment>
 </net>
@@
 </segment>
 <segment>
-<pinref part="JP2" gate="A" pin="6"/>
-<wire x1="127" y1="63.5" x2="134.62" y2="63.5" width="0.1524" layer="91"/>
-<label x="127" y="63.5" size="1.778" layer="95" rot="MR0"/>
+<wire x1="101.6" y1="76.2" x2="109.22" y2="76.2" width="0.1524" layer="91"/>
+<label x="101.6" y="76.2" size="1.778" layer="95" rot="MR0"/>
+<pinref part="U$3" gate="G$1" pin="VDD"/>
 </segment>
 </net>
@@
 </segment>
 </net>
-<net name="GIO1" class="0">
-<segment>
-<pinref part="JP1" gate="A" pin="2"/>
-<wire x1="114.3" y1="73.66" x2="106.68" y2="73.66" width="0.1524" layer="91"/>
-<label x="106.68" y="73.66" size="1.778" layer="95" rot="MR0"/>
-</segment>
-</net>
-<net name="GIO2" class="0">
-<segment>
-<pinref part="JP1" gate="A" pin="4"/>
-<wire x1="106.68" y1="68.58" x2="114.3" y2="68.58" width="0.1524" layer="91"/>
-<label x="106.68" y="68.58" size="1.778" layer="95" rot="MR0"/>
-</segment>
-</net>
 <net name="SDIO" class="0">
-<segment>
-<pinref part="JP2" gate="A" pin="1"/>
-<wire x1="127" y1="76.2" x2="134.62" y2="76.2" width="0.1524" layer="91"/>
-<label x="127" y="76.2" size="1.778" layer="95" rot="MR0"/>
-</segment>
 <segment>
 <pinref part="U$1" gate="G$1" pin="5"/>
@@
 <label x="60.96" y="20.32" size="1.778" layer="95"/>
 </segment>
+<segment>
+<pinref part="U$3" gate="G$1" pin="SDIO"/>
+<wire x1="147.32" y1="76.2" x2="139.7" y2="76.2" width="0.1524" layer="91"/>
+<label x="147.32" y="76.2" size="1.778" layer="95"/>
+</segment>
 </net>
 <net name="SCK" class="0">
-<segment>
-<pinref part="JP2" gate="A" pin="2"/>
-<wire x1="127" y1="73.66" x2="134.62" y2="73.66" width="0.1524" layer="91"/>
-<label x="127" y="73.66" size="1.778" layer="95" rot="MR0"/>
-</segment>
 <segment>
 <pinref part="J3" gate="G$1" pin="6"/>
@@
 <label x="60.96" y="22.86" size="1.778" layer="95"/>
 </segment>
+<segment>
+<pinref part="U$3" gate="G$1" pin="SCK"/>
+<wire x1="147.32" y1="73.66" x2="139.7" y2="73.66" width="0.1524" layer="91"/>
+<label x="147.32" y="73.66" size="1.778" layer="95"/>
+</segment>
 </net>
 <net name="SCS" class="0">
-<segment>
-<pinref part="JP2" gate="A" pin="3"/>
-<wire x1="127" y1="71.12" x2="134.62" y2="71.12" width="0.1524" layer="91"/>
-<label x="127" y="71.12" size="1.778" layer="95" rot="MR0"/>
-</segment>
 <segment>
 <pinref part="J3" gate="G$1" pin="8"/>
@@
 <label x="60.96" y="27.94" size="1.778" layer="95"/>
 </segment>
-</net>
+<segment>
+<pinref part="U$3" gate="G$1" pin="SCS"/>
+<wire x1="147.32" y1="71.12" x2="139.7" y2="71.12" width="0.1524" layer="91"/>
+<label x="147.32" y="71.12" size="1.778" layer="95"/>
+</segment>
+</net>
+<net name="GIO1" class="0">
+<segment>
+<pinref part="U$3" gate="G$1" pin="GIO1"/>
+<wire x1="147.32" y1="68.58" x2="139.7" y2="68.58" width="0.1524" layer="91"/>
+<label x="147.32" y="68.58" size="1.778" layer="95"/>
+</segment>
+</net>
+<net name="GIO2" class="0">
+<segment>
+<pinref part="U$3" gate="G$1" pin="GIO2"/>
+<wire x1="147.32" y1="66.04" x2="139.7" y2="66.04" width="0.1524" layer="91"/>
+<label x="147.32" y="66.04" size="1.778" layer="95"/>
+</segment>
+</net>
